File: Kronos V1/WS2812B 2020 Array.kicad_sch (KiCad schematic)
At the start: 166 parts, among them U12 WS2812-2020, U13 WS2812-2020, U14 WS2812-2020, U15 WS2812-2020, U16 WS2812-2020, U17 WS2812-2020, U18 WS2812-2020, U19 WS2812-2020, U20 WS2812-2020, U21 WS2812-2020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

Commit message: Corrected error with H4 ARGB
Connections:
- net at U92.1 (DO): no longer U91.1 (DO)
- net at U92.3 (DI): now also U91.1 (DO)
